Commit message: Rebase from 'upstream'

File: models/simple_humanoid.urdf (robot description, URDF)
Before this commit: robot simple_humanoid, 30 links, 29 joints
Links:
- link WAIST_LINK0: geometry collision cylinder length=1 radius=1; collision mesh filename=package://simple_humanoid_description/box.stl
